File: harduino0.2.brd (EAGLE design)
At the start: 23 parts, among them IC1 ATMEGA48/88/168-AU, IC3 7805DT, J1 1X2-3.5MM

Commit message: harduino
update 0.2
Parts:
- removed C6: 22pf, 01_SparkFun:1206
- added C1: 10uf, ng:1206
- C2: value 10uf -> .1uf
- C3: value .1uf -> 1uf
- C4: value 1uf -> 22pf; device ng:1206 -> 01_SparkFun:1206
- R3, R4: value (none) -> 499
- moved C4 18.1 mm to (21.1, 37.1), turned to 270 degrees
- moved C2 17.2 mm to (24.7, 51.3)
- moved C5 4.34 mm to (25.5, 37.0)
- moved C3 3.45 mm to (24.7, 54.8), turned to 0 degrees
- renumbered IC3 to IC2, LED to D1, U$1 to D2, U$2 to D3
Connections:
- net BATT: now also C1.2; no longer C2.2
- net DTR: now also C2.2; no longer C3.2
- net GND: now also C1.1, C3.1; no longer C2.1, C6.1
- net N$1: now also C5.2; no longer C6.2
- net N$2: now also C4.2; no longer C5.2
- net RST: now also C2.1; no longer C3.1
- net VCC: now also C3.2; no longer C4.2
Changed lines of the file:
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@@
 <?xml version="1.0" encoding="utf-8"?>
 <!DOCTYPE eagle SYSTEM "eagle.dtd">
-<eagle version="7.4.0">
+<eagle version="7.5.0">
 <drawing>
 <settings>
@@
 <element name="S1" library="ng" package="6MM_SWITCH" value="" x="26.2128" y="8.5852"/>
 <element name="R2" library="ng" package="1206" value="499" x="16.8656" y="14.3002" rot="R180"/>
-<element name="LED" library="ng" package="1206" value="" x="16.8656" y="10.6426"/>
-<element name="C2" library="ng" package="1206" value="10uf" x="41.5798" y="48.2092" rot="R180"/>
-<element name="C3" library="ng" package="1206" value=".1uf" x="24.6634" y="51.308" rot="R180"/>
-<element name="C4" library="ng" package="1206" value="1uf" x="24.6634" y="54.7624"/>
+<element name="D1" library="ng" package="1206" value="" x="16.8656" y="10.6426"/>
+<element name="C1" library="ng" package="1206" value="10uf" x="41.5798" y="48.2092" rot="R180"/>
+<element name="C2" library="ng" package="1206" value=".1uf" x="24.6634" y="51.308" rot="R180"/>
+<element name="C3" library="ng" package="1206" value="1uf" x="24.6634" y="54.7624"/>
 <element name="ISP" library="SparkFun" package="1X06-SMD" value="" x="13.5636" y="58.5216" rot="R180"/>
-<element name="C5" library="01_SparkFun" package="1206" value="22pf" x="21.1074" y="37.0586" rot="R270"/>
-<element name="C6" library="01_SparkFun" package="1206" value="22pf" x="25.4508" y="36.9824" rot="R270"/>
+<element name="C4" library="01_SparkFun" package="1206" value="22pf" x="21.1074" y="37.0586" rot="R270"/>
+<element name="C5" library="01_SparkFun" package="1206" value="22pf" x="25.4508" y="36.9824" rot="R270"/>
 <element name="XTAL" library="01_ng" package="CS10" value="16mhz" x="23.3426" y="31.4452"/>
 <element name="JP1" library="01_SparkFun" package="1X06_LONGPADS" value="" x="37.0586" y="9.1186" rot="R90"/>
@@
 <element name="J1" library="01_adafruit" package="3.5MMTERM" value="1X2-3.5MM" x="35.2298" y="63.2968"/>
 <element name="JP5" library="01_SparkFun" package="1X02_LONGPADS" value="" x="37.0586" y="39.6748" rot="R90"/>
-<element name="U$1" library="01_FAB_Hello" package="1206" value="" x="18.5166" y="44.4246" rot="R180"/>
-<element name="U$2" library="01_FAB_Hello" package="1206" value="" x="18.4658" y="47.5234" rot="R180"/>
-<element name="R3" library="01_FAB_Hello" package="1206" value="" x="24.511" y="44.4754" rot="R180"/>
-<element name="R4" library="01_FAB_Hello" package="1206" value="" x="24.5618" y="47.5234" rot="R180"/>
-<element name="IC3" library="01_adafruit" package="TO252" value="7805DT" x="35.052" y="52.6034"/>
+<element name="D2" library="01_FAB_Hello" package="1206" value="" x="18.5166" y="44.4246" rot="R180"/>
+<element name="D3" library="01_FAB_Hello" package="1206" value="" x="18.4658" y="47.5234" rot="R180"/>
+<element name="R3" library="01_FAB_Hello" package="1206" value="499" x="24.511" y="44.4754" rot="R180"/>
+<element name="R4" library="01_FAB_Hello" package="1206" value="499" x="24.5618" y="47.5234" rot="R180"/>
+<element name="IC2" library="01_adafruit" package="TO252" value="7805DT" x="35.052" y="52.6034"/>
 </elements>
 <signals>
 <signal name="GND">
 <contactref element="IC1" pad="21"/>
-<contactref element="LED" pad="2"/>
-<contactref element="C4" pad="1"/>
+<contactref element="D1" pad="2"/>
+<contactref element="C3" pad="1"/>
 <contactref element="IC1" pad="5"/>
 <contactref element="ISP" pad="2"/>
 <contactref element="ISP" pad="1"/>
-<contactref element="C6" pad="1"/>
 <contactref element="C5" pad="1"/>
+<contactref element="C4" pad="1"/>
 <contactref element="S1" pad="2"/>
 <contactref element="S1" pad="1"/>
@@
 <wire x1="19.9136" y1="53.5216" x2="21.4122" y2="53.5216" width="0.4064" layer="1"/>
 <wire x1="21.4122" y1="53.5216" x2="21.4122" y2="61.087" width="0.4064" layer="1"/>
-<contactref element="IC3" pad="3"/>
-<contactref element="C2" pad="1"/>
+<contactref element="IC2" pad="3"/>
+<contactref element="C1" pad="1"/>
 <contactref element="J1" pad="2"/>
 <polygon width="0.4064" layer="1" isolate="1.016">
@@
 <contactref element="IC1" pad="4"/>
 <contactref element="R1" pad="2"/>
-<contactref element="C4" pad="2"/>
+<contactref element="C3" pad="2"/>
 <contactref element="ISP" pad="3"/>
 <contactref element="IC1" pad="6"/>
@@
 <wire x1="26.0854" y1="54.7624" x2="26.0862" y2="53.1114" width="0.4064" layer="1"/>
 <wire x1="26.0862" y1="53.1114" x2="24.6634" y2="53.1114" width="0.4064" layer="1"/>
-<contactref element="IC3" pad="1"/>
+<contactref element="IC2" pad="1"/>
 <wire x1="32.772" y1="47.8034" x2="29.972" y2="47.8034" width="0.3556" layer="1"/>
 <wire x1="29.972" y1="47.8034" x2="29.972" y2="54.864" width="0.3556" layer="1"/>
@@
 <contactref element="DIST" pad="1"/>
 <wire x1="33.8836" y1="24.3586" x2="37.0586" y2="24.3586" width="0.4064" layer="1"/>
-<contactref element="C3" pad="1"/>
+<contactref element="C2" pad="1"/>
 <wire x1="26.0854" y1="51.308" x2="28.956" y2="51.308" width="0.3556" layer="1"/>
 <wire x1="28.956" y1="51.308" x2="28.956" y2="46.228" width="0.3556" layer="1"/>
@@
 <signal name="N$23">
 <contactref element="R2" pad="2"/>
-<contactref element="LED" pad="1"/>
+<contactref element="D1" pad="1"/>
 <wire x1="15.4436" y1="10.6426" x2="15.4436" y2="14.3002" width="0.3556" layer="1"/>
 </signal>
 <signal name="DTR">
 <contactref element="ISP" pad="6"/>
-<contactref element="C3" pad="2"/>
+<contactref element="C2" pad="2"/>
 <wire x1="7.2136" y1="53.5216" x2="7.2136" y2="57.1246" width="0.4064" layer="1"/>
 <wire x1="7.2136" y1="57.1246" x2="16.0782" y2="57.1246" width="0.4064" layer="1"/>
@@
 <contactref element="ISP" pad="5"/>
 <wire x1="9.9568" y1="54.563" x2="9.7536" y2="53.5216" width="0.4064" layer="1"/>
-<contactref element="U$1" pad="2"/>
+<contactref element="D2" pad="2"/>
 <wire x1="9.7536" y1="53.5216" x2="9.7536" y2="43.815" width="0.3556" layer="1"/>
 <wire x1="9.7536" y1="43.815" x2="16.51" y2="43.815" width="0.3556" layer="1"/>
@@
 <contactref element="ISP" pad="4"/>
 <wire x1="12.2936" y1="53.5216" x2="12.2936" y2="46.863" width="0.3556" layer="1"/>
-<contactref element="U$2" pad="2"/>
+<contactref element="D3" pad="2"/>
 <wire x1="12.2936" y1="46.863" x2="17.145" y2="46.863" width="0.3556" layer="1"/>
 <wire x1="17.145" y1="46.863" x2="17.145" y2="47.0154" width="0.3556" layer="1"/>
@@
 <contactref element="IC1" pad="7"/>
 <contactref element="XTAL" pad="P$2"/>
-<contactref element="C6" pad="2"/>
+<contactref element="C5" pad="2"/>
 <wire x1="21.9014" y1="24.8412" x2="21.9014" y2="29.0576" width="0.4064" layer="1"/>
 <wire x1="21.9014" y1="29.0576" x2="25.9588" y2="29.0576" width="0.4064" layer="1"/>
@@
 <contactref element="IC1" pad="8"/>
 <contactref element="XTAL" pad="P$1"/>
-<contactref element="C5" pad="2"/>
+<contactref element="C4" pad="2"/>
 <wire x1="21.1014" y1="25.0952" x2="21.1014" y2="31.1912" width="0.4064" layer="1"/>
 <wire x1="21.1014" y1="31.1912" x2="21.0566" y2="31.4452" width="0.4064" layer="1"/>
@@
 <signal name="BATT">
 <contactref element="J1" pad="1"/>
-<contactref element="IC3" pad="2"/>
-<contactref element="C2" pad="2"/>
+<contactref element="IC2" pad="2"/>
+<contactref element="C1" pad="2"/>
 <wire x1="37.332" y1="47.8034" x2="37.586" y2="48.2092" width="1.016" layer="1"/>
 <wire x1="40.1578" y1="48.2092" x2="40.132" y2="48.0318" width="1.016" layer="1"/>
@@
 <signal name="N$19">
 <contactref element="R4" pad="2"/>
-<contactref element="U$2" pad="1"/>
+<contactref element="D3" pad="1"/>
 <wire x1="19.8878" y1="47.5234" x2="19.8878" y2="46.863" width="0.3556" layer="1"/>
 <wire x1="19.8878" y1="46.863" x2="23.495" y2="46.863" width="0.3556" layer="1"/>
@@
 </signal>
 <signal name="N$21">
-<contactref element="U$1" pad="1"/>
+<contactref element="D2" pad="1"/>
 <contactref element="R3" pad="2"/>
 <wire x1="23.089" y1="44.4754" x2="23.343" y2="44.4246" width="0.3556" layer="1"/>
