File: harduino0.2.sch (EAGLE design)
At the start: 23 parts, among them IC1 ATMEGA48/88/168-AU, IC3 7805DT, J1 1X2-3.5MM

Commit message: harduino
update 0.2
Parts:
- removed C6: 22pf, 01_SparkFun:CAP1206
- added C1: 10uf, ng:UNPOLARIZED_CAPACITOR1206
- C2: value 10uf -> .1uf
- C3: value .1uf -> 1uf
- C4: value 1uf -> 22pf; device ng:UNPOLARIZED_CAPACITOR1206 -> 01_SparkFun:CAP1206
- R3, R4: value (none) -> 499
- renumbered IC3 to IC2, LED to D1, U$1 to D2, U$2 to D3
Connections:
- net BATT: now also C1.2; no longer C2.2
- net DTR: now also C2.2; no longer C3.2
- net GND: now also C1.1, C3.1; no longer C2.1, C6.1
- net N$1: now also C5.2; no longer C6.2
- net N$2: now also C4.2; no longer C5.2
- net RST: now also C2.1; no longer C3.1
- net VCC: now also C3.2; no longer C4.2
Other:
- moved on the sheet: C2, C3, C5
Changed lines of the file:
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@@
 <?xml version="1.0" encoding="utf-8"?>
 <!DOCTYPE eagle SYSTEM "eagle.dtd">
-<eagle version="7.4.0">
+<eagle version="7.5.0">
 <drawing>
 <settings>
@@
 <part name="S1" library="ng" deviceset="6MM_SWITCH" device="6MM_SWITCH"/>
 <part name="R2" library="ng" deviceset="RESISTOR" device="1206" value="499"/>
-<part name="LED" library="ng" deviceset="LED" device="1206"/>
+<part name="D1" library="ng" deviceset="LED" device="1206"/>
 <part name="GND3" library="supply1" deviceset="GND" device=""/>
-<part name="C2" library="ng" deviceset="UNPOLARIZED_CAPACITOR" device="1206" value="10uf"/>
-<part name="C3" library="ng" deviceset="UNPOLARIZED_CAPACITOR" device="1206" value=".1uf"/>
+<part name="C1" library="ng" deviceset="UNPOLARIZED_CAPACITOR" device="1206" value="10uf"/>
+<part name="C2" library="ng" deviceset="UNPOLARIZED_CAPACITOR" device="1206" value=".1uf"/>
 <part name="P+4" library="supply1" deviceset="VCC" device=""/>
 <part name="GND5" library="supply1" deviceset="GND" device=""/>
 <part name="GND6" library="supply1" deviceset="GND" device=""/>
-<part name="C4" library="ng" deviceset="UNPOLARIZED_CAPACITOR" device="1206" value="1uf"/>
+<part name="C3" library="ng" deviceset="UNPOLARIZED_CAPACITOR" device="1206" value="1uf"/>
 <part name="ISP" library="SparkFun" deviceset="M06" device="SMD"/>
+<part name="C4" library="01_SparkFun" deviceset="CAP" device="1206" value="22pf"/>
 <part name="C5" library="01_SparkFun" deviceset="CAP" device="1206" value="22pf"/>
-<part name="C6" library="01_SparkFun" deviceset="CAP" device="1206" value="22pf"/>
 <part name="XTAL" library="01_ng" deviceset="CRYSTAL" device="CS10" value="16mhz"/>
 <part name="JP1" library="01_SparkFun" deviceset="M06" device="LONGPADS"/>
@@
 <part name="J1" library="01_adafruit" deviceset="1X2" device="-3.5MM"/>
 <part name="JP5" library="01_SparkFun" deviceset="M02" device=""/>
-<part name="U$1" library="01_FAB_Hello" deviceset="LED" device="1206"/>
-<part name="U$2" library="01_FAB_Hello" deviceset="LED" device="1206"/>
-<part name="R3" library="01_FAB_Hello" deviceset="RESISTOR" device="1206"/>
-<part name="R4" library="01_FAB_Hello" deviceset="RESISTOR" device="1206"/>
-<part name="IC3" library="01_adafruit" deviceset="78*" device="DT" technology="05"/>
+<part name="D2" library="01_FAB_Hello" deviceset="LED" device="1206"/>
+<part name="D3" library="01_FAB_Hello" deviceset="LED" device="1206"/>
+<part name="R3" library="01_FAB_Hello" deviceset="RESISTOR" device="1206" value="499"/>
+<part name="R4" library="01_FAB_Hello" deviceset="RESISTOR" device="1206" value="499"/>
+<part name="IC2" library="01_adafruit" deviceset="78*" device="DT" technology="05"/>
 </parts>
 <sheets>
@@
 <instance part="S1" gate="2" x="-40.64" y="73.66"/>
 <instance part="R2" gate="G$1" x="96.52" y="-5.08"/>
-<instance part="LED" gate="G$1" x="109.22" y="-5.08" rot="R90"/>
+<instance part="D1" gate="G$1" x="109.22" y="-5.08" rot="R90"/>
 <instance part="GND3" gate="1" x="116.84" y="-5.08" rot="R90"/>
-<instance part="C2" gate="1" x="-110.49" y="99.06" rot="R90"/>
-<instance part="C3" gate="1" x="-22.86" y="83.82" rot="R90"/>
+<instance part="C1" gate="1" x="-110.49" y="99.06" rot="R90"/>
+<instance part="C2" gate="1" x="-22.86" y="83.82" rot="R90"/>
 <instance part="P+4" gate="VCC" x="-78.74" y="53.34"/>
 <instance part="GND5" gate="1" x="-78.74" y="33.02"/>
 <instance part="GND6" gate="1" x="-40.64" y="58.42"/>
-<instance part="C4" gate="1" x="-78.74" y="43.18" rot="R90"/>
+<instance part="C3" gate="1" x="-78.74" y="43.18" rot="R90"/>
 <instance part="ISP" gate="G$1" x="157.48" y="114.3" rot="MR0"/>
-<instance part="C5" gate="G$1" x="-10.16" y="57.15" rot="R90"/>
-<instance part="C6" gate="G$1" x="-10.16" y="64.77" rot="R90"/>
+<instance part="C4" gate="G$1" x="-10.16" y="57.15" rot="R90"/>
+<instance part="C5" gate="G$1" x="-10.16" y="64.77" rot="R90"/>
 <instance part="XTAL" gate="G$1" x="0" y="60.96" rot="R90"/>
 <instance part="JP1" gate="G$1" x="97.79" y="73.66" rot="R180"/>
@@
 <instance part="J1" gate="G$1" x="-92.71" y="99.06"/>
 <instance part="JP5" gate="G$1" x="101.6" y="93.98" rot="R180"/>
-<instance part="U$1" gate="G$1" x="120.65" y="121.92" rot="R90"/>
-<instance part="U$2" gate="G$1" x="120.65" y="114.3" rot="R90"/>
+<instance part="D2" gate="G$1" x="120.65" y="121.92" rot="R90"/>
+<instance part="D3" gate="G$1" x="120.65" y="114.3" rot="R90"/>
 <instance part="R3" gate="G$1" x="107.95" y="121.92"/>
 <instance part="R4" gate="G$1" x="107.95" y="114.3"/>
-<instance part="IC3" gate="A1" x="-129.54" y="101.6"/>
+<instance part="IC2" gate="A1" x="-129.54" y="101.6"/>
 </instances>
 <busses>
@@
 <wire x1="-78.74" y1="50.8" x2="-78.74" y2="45.72" width="0.1524" layer="91"/>
 <pinref part="P+4" gate="VCC" pin="VCC"/>
-<pinref part="C4" gate="1" pin="2"/>
+<pinref part="C3" gate="1" pin="2"/>
 </segment>
 <segment>
@@
 <wire x1="-139.7" y1="101.6" x2="-146.05" y2="101.6" width="0.1524" layer="91"/>
 <label x="-146.05" y="101.6" size="1.778" layer="95" rot="R180"/>
-<pinref part="IC3" gate="A1" pin="VI"/>
+<pinref part="IC2" gate="A1" pin="VI"/>
 </segment>
 <segment>
@@
 <pinref part="IC1" gate="1" pin="PC6(/RESET/PCINT14)"/>
 <pinref part="S1" gate="2" pin="S1"/>
-<pinref part="C3" gate="1" pin="1"/>
+<pinref part="C2" gate="1" pin="1"/>
 <wire x1="-22.86" y1="78.74" x2="-38.1" y2="78.74" width="0.1524" layer="91"/>
 <junction x="-22.86" y="78.74"/>
@@
 <segment>
 <wire x1="111.76" y1="-5.08" x2="114.3" y2="-5.08" width="0.1524" layer="91"/>
-<pinref part="LED" gate="G$1" pin="C"/>
+<pinref part="D1" gate="G$1" pin="C"/>
 <pinref part="GND3" gate="1" pin="GND"/>
 </segment>
@@
 <wire x1="-78.74" y1="38.1" x2="-78.74" y2="35.56" width="0.1524" layer="91"/>
 <pinref part="GND5" gate="1" pin="GND"/>
-<pinref part="C4" gate="1" pin="1"/>
+<pinref part="C3" gate="1" pin="1"/>
 </segment>
 <segment>
@@
 </segment>
 <segment>
-<pinref part="C6" gate="G$1" pin="1"/>
+<pinref part="C5" gate="G$1" pin="1"/>
 <wire x1="-15.24" y1="64.77" x2="-17.78" y2="64.77" width="0.1524" layer="91"/>
 <label x="-17.78" y="64.77" size="1.27" layer="95" rot="R180" xref="yes"/>
 </segment>
 <segment>
-<pinref part="C5" gate="G$1" pin="1"/>
+<pinref part="C4" gate="G$1" pin="1"/>
 <wire x1="-15.24" y1="57.15" x2="-17.78" y2="57.15" width="0.1524" layer="91"/>
 <label x="-17.78" y="57.15" size="1.27" layer="95" rot="R180" xref="yes"/>
@@
 <wire x1="-129.54" y1="93.98" x2="-129.54" y2="91.44" width="0.1524" layer="91"/>
 <wire x1="-129.54" y1="93.98" x2="-110.49" y2="93.98" width="0.1524" layer="91"/>
-<pinref part="IC3" gate="A1" pin="GND"/>
-<pinref part="C2" gate="1" pin="1"/>
+<pinref part="IC2" gate="A1" pin="GND"/>
+<pinref part="C1" gate="1" pin="1"/>
 <pinref part="J1" gate="G$1" pin="2"/>
 <wire x1="-102.87" y1="99.06" x2="-97.79" y2="99.06" width="0.1524" layer="91"/>
@@
 <wire x1="101.6" y1="-5.08" x2="104.14" y2="-5.08" width="0.1524" layer="91"/>
 <pinref part="R2" gate="G$1" pin="2"/>
-<pinref part="LED" gate="G$1" pin="A"/>
+<pinref part="D1" gate="G$1" pin="A"/>
 </segment>
 </net>
@@
 </segment>
 <segment>
-<pinref part="C3" gate="1" pin="2"/>
+<pinref part="C2" gate="1" pin="2"/>
 <wire x1="-22.86" y1="86.36" x2="-22.86" y2="96.52" width="0.1524" layer="91"/>
 <label x="-22.86" y="96.52" size="1.778" layer="95" rot="R180"/>
@@
 <label x="147.32" y="119.38" size="1.778" layer="95" rot="R180"/>
 <pinref part="ISP" gate="G$1" pin="5"/>
-<pinref part="U$1" gate="G$1" pin="C"/>
+<pinref part="D2" gate="G$1" pin="C"/>
 <wire x1="123.19" y1="121.92" x2="134.62" y2="121.92" width="0.1524" layer="91"/>
 <wire x1="134.62" y1="121.92" x2="134.62" y2="119.38" width="0.1524" layer="91"/>
@@
 <wire x1="152.4" y1="116.84" x2="134.62" y2="116.84" width="0.1524" layer="91"/>
 <wire x1="134.62" y1="116.84" x2="134.62" y2="114.3" width="0.1524" layer="91"/>
-<pinref part="U$2" gate="G$1" pin="C"/>
+<pinref part="D3" gate="G$1" pin="C"/>
 <wire x1="134.62" y1="114.3" x2="123.19" y2="114.3" width="0.1524" layer="91"/>
 </segment>
@@
 <wire x1="10.16" y1="64.77" x2="0" y2="64.77" width="0.1524" layer="91"/>
 <wire x1="0" y1="64.77" x2="-7.62" y2="64.77" width="0.1524" layer="91"/>
-<pinref part="C6" gate="G$1" pin="2"/>
+<pinref part="C5" gate="G$1" pin="2"/>
 </segment>
 </net>
@@
 <wire x1="10.16" y1="57.15" x2="0" y2="57.15" width="0.1524" layer="91"/>
 <wire x1="0" y1="57.15" x2="-7.62" y2="57.15" width="0.1524" layer="91"/>
-<pinref part="C5" gate="G$1" pin="2"/>
+<pinref part="C4" gate="G$1" pin="2"/>
 </segment>
 </net>
@@
 <label x="-114.3" y="101.6" size="1.778" layer="95"/>
 <pinref part="J1" gate="G$1" pin="1"/>
-<pinref part="IC3" gate="A1" pin="VO"/>
-<pinref part="C2" gate="1" pin="2"/>
+<pinref part="IC2" gate="A1" pin="VO"/>
+<pinref part="C1" gate="1" pin="2"/>
 <wire x1="-110.49" y1="101.6" x2="-97.79" y2="101.6" width="0.1524" layer="91"/>
 </segment>
@@
 <net name="N$19" class="0">
 <segment>
-<pinref part="U$2" gate="G$1" pin="A"/>
+<pinref part="D3" gate="G$1" pin="A"/>
 <pinref part="R4" gate="G$1" pin="2"/>
 <wire x1="113.03" y1="114.3" x2="115.57" y2="114.3" width="0.1524" layer="91"/>
@@
 <net name="N$21" class="0">
 <segment>
-<pinref part="U$1" gate="G$1" pin="A"/>
+<pinref part="D2" gate="G$1" pin="A"/>
 <pinref part="R3" gate="G$1" pin="2"/>
 <wire x1="113.03" y1="121.92" x2="115.57" y2="121.92" width="0.1524" layer="91"/>
